File: switch-test-board/switch-test-board.kicad_pcb (KiCad board)
At the start: 4 copper layers, 100.7 x 102.7 mm, 201 parts, among them J1 USB_B_Micro, J2 2011-2X10G00SD025B, J3 1367073-1, J4 2011-2X10G00SD025B, SW1 PTS645SM43SMTR92 LFS, U1 RPI4CM, U10 MDT420M02001, U2 KSZ9477S, U3 LD39200PUR, U4 piSlice-PCIe-X1-Conn, U5 LM1085ISX-3.3/NOPB, U6 LD39200PUR, U7 LD39200PUR, U8 piSlice-PCIe-X1-Edge, U9 MIC826TYMT, Y1 ABM8G-25.000MHZ-B4Y-T

Commit message: PCB updated.
Parts:
- removed C45: 10uF, Capacitor_SMD:C_0603_1608Metric
- removed FB3: BLM18EG221SN1D, kicad-lib:ferrite-blm18
- added C100: 0.1uF, Capacitor_SMD:C_0402_1005Metric, F.Cu at (80.6, 113.5)
- added C101: 0.1uF, Capacitor_SMD:C_0402_1005Metric, F.Cu at (97.3, 113.4)
- added C102: 0.1uF, Capacitor_SMD:C_0402_1005Metric, F.Cu at (96.3, 113.4)
- added C99: 0.1uF, Capacitor_SMD:C_0402_1005Metric, F.Cu at (81.6, 113.5)
- added FB8: BLM18EG221SN1D, kicad-lib:ferrite-blm18, F.Cu at (99.7, 140.1)
- added J5: JK0654219, Connector_RJ:RJ45_Pulse_JK0654219NL_Horizontal, F.Cu at (93.9, 122.3)
- C77, C80, R54, TP7, TP8, U10: moved to B.Cu
- moved R54 234.2 mm to (156.9, 84.0), turned to 180 degrees
- moved TP8 231.8 mm to (160.0, 96.0)
- moved TP7 224.0 mm to (171.0, 96.0)
- moved D4 210.6 mm to (139.7, 101.9), turned to 270 degrees
- moved R13 209.0 mm to (139.6, 99.4), turned to 270 degrees
- moved D3 208.5 mm to (138.0, 101.9), turned to 270 degrees
- moved R12 204.7 mm to (140.8, 99.4), turned to 270 degrees
- moved D2 202.0 mm to (141.4, 101.9), turned to 270 degrees
- moved R11 201.4 mm to (141.9, 99.4), turned to 270 degrees
- moved C7 193.4 mm to (142.6, 109.5), turned to 180 degrees
- moved TP3 192.0 mm to (180.8, 144.4)
- moved C6 190.8 mm to (142.6, 111.0), turned to 180 degrees
- moved C5 188.7 mm to (142.6, 112.5), turned to 180 degrees
- moved TP2 187.3 mm to (174.3, 147.2)
- moved C4 185.8 mm to (142.6, 114.0), turned to 180 degrees
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Connections:
- net /RPI_USB_DM renamed /RPI_USBD_N
- net /RPI_USB_DP renamed /RPI_USBD_P
- C60 pad 1: /DVDDL_1V2 -> +1V2
- C62 pad 1: /DVDDL_1V2 -> +1V2
- C64 pad 1: /DVDDL_1V2 -> +1V2
- C69 pad 1: /DVDDL_1V2 -> +1V2
- C74 pad 1: /DVDDL_1V2 -> +1V2
- C79 pad 1: /DVDDL_1V2 -> +1V2
- C82 pad 1: /DVDDL_1V2 -> +1V2
- C85 pad 1: /DVDDL_1V2 -> +1V2
- C88 pad 1: /DVDDL_1V2 -> +1V2
- C91 pad 1: /DVDDL_1V2 -> +1V2
- U2 pad 104: /DVDDL_1V2 -> +1V2
- U2 pad 11: /DVDDL_1V2 -> +1V2
- U2 pad 110: /DVDDL_1V2 -> +1V2
- U2 pad 23: /DVDDL_1V2 -> +1V2
- U2 pad 34: Net-(U2-Pad34) -> /P4_TXRX_A_P
- U2 pad 35: Net-(U2-Pad35) -> /P4_TXRX_A_N
- U2 pad 37: Net-(U2-Pad37) -> /P4_TXRX_B_P
- U2 pad 38: Net-(U2-Pad38) -> /P4_TXRX_B_N
- U2 pad 39: Net-(U2-Pad39) -> /P4_TXRX_C_P
- U2 pad 40: Net-(U2-Pad40) -> /P4_TXRX_C_N
- U2 pad 42: Net-(U2-Pad42) -> /P4_TXRX_D_P
- U2 pad 43: Net-(U2-Pad43) -> /P4_TXRX_D_N
- U2 pad 45: /DVDDL_1V2 -> +1V2
- U2 pad 56: /DVDDL_1V2 -> +1V2
- U2 pad 66: /DVDDL_1V2 -> +1V2
- U2 pad 70: /DVDDL_1V2 -> +1V2
- U2 pad 87: /DVDDL_1V2 -> +1V2
Routing:
- net +5V: track 0.00 -> 143.2 mm, vias 0 -> 12
- net +2V5: track 0.00 -> 105.8 mm, vias 0 -> 13
- net +1V2: track 0.00 -> 96.4 mm, vias 0 -> 26
- net /RPI_PCIe_CLK_nREQ: track 0.00 -> 39.6 mm, vias 0 -> 1
- net /RPI_PCIe_CLK_P: track 0.00 -> 36.0 mm, vias 0 -> 1
- net /RPI_PCIe_CLK_N: track 0.00 -> 35.5 mm, vias 0 -> 1
- net /P4_TXRX_B_P: track 0.00 -> 35.4 mm, vias 0 -> 1
- net /P4_TXRX_B_N: track 0.00 -> 35.4 mm, vias 0 -> 1
- net /P4_TXRX_A_P: track 0.00 -> 34.1 mm
- net /RPI_PCIe_TX_P: track 0.00 -> 33.9 mm, vias 0 -> 1
- net /P4_TXRX_A_N: track 0.00 -> 33.6 mm
- net /RPI_PCIe_TX_N: track 0.00 -> 33.4 mm, vias 0 -> 1
- net /P4_TXRX_C_P: track 0.00 -> 32.6 mm
- net /P4_TXRX_C_N: track 0.00 -> 32.2 mm
- net /RPI_PCIe_RX_P: track 0.00 -> 31.9 mm, vias 0 -> 1
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- added copper zone on F.Cu, net (none)
- added copper zone on F.Cu, net +1V2
- added copper zone on In2.Cu, net +1V2
- added copper zone on F.Cu, net +2V5
- added copper zone on F.Cu, net +3V3
- added copper zone on F.Cu, net +5V
- added copper zone on F.Cu, net /3V3_PCIE
- added copper zone on B.Cu, net /AVDDH_2V5
- added copper zone on F.Cu, net /AVDDL_1V2
- added copper zone on In2.Cu, net /AVDDL_1V2
- added copper zone on F.Cu, net GND
- added copper zone on B.Cu, net GNDREF
Other:
- board size 100.7 x 102.7 mm -> 114.4 x 102.7 mm
- net class PCIe: clearance 0.1 -> 0.1524; trace_width 0.1 -> 0.14097
- net class USB: clearance 0.1 -> 0.1524; trace_width 0.1 -> 0.14097

Commit message: PCB Design Completed.
Parts:
- removed C49: 0.1uF, Capacitor_SMD:C_0402_1005Metric
- removed C50, C54: 10uF, Capacitor_SMD:C_0603_1608Metric
- removed J4: 2011-2X10G00SD025B, Connector_PinHeader_2.54mm:PinHeader_2x10_P2.54mm_Vertical
- removed R22: 22R, Resistor_SMD:R_0402_1005Metric
- removed R30: 56K, Resistor_SMD:R_0402_1005Metric
- removed R31: 10K, Resistor_SMD:R_0402_1005Metric
- removed TP4: TestPoint, TestPoint:TestPoint_Pad_D1.0mm
- removed U3: LD39200PUR, Package_DFN_QFN:DFN-6-1EP_3x3mm_P0.95mm_EP1.7x2.6mm
- added R56: 0R_DNP, Resistor_SMD:R_0402_1005Metric, F.Cu at (105.2, 124.8)
- added R57: 0R_DNP, Resistor_SMD:R_0402_1005Metric, F.Cu at (105.3, 117.0)
- added R58: 0R_DNP, Resistor_SMD:R_0402_1005Metric, F.Cu at (139.9, 119.5)
- added R59: 0R_DNP, Resistor_SMD:R_0402_1005Metric, F.Cu at (139.9, 123.3)
- added R60: 0R_DNP, Resistor_SMD:R_0402_1005Metric, F.Cu at (138.1, 109.8)
- added R61: 0R_DNP, Resistor_SMD:R_0402_1005Metric, F.Cu at (138.1, 107.0)
- added R62: 0R_DNP, Resistor_SMD:R_0402_1005Metric, F.Cu at (139.9, 117.6)
- added R63: 0R_DNP, Resistor_SMD:R_0402_1005Metric, F.Cu at (139.9, 121.4)
- added R64: 0R_DNP, Resistor_SMD:R_0402_1005Metric, F.Cu at (138.1, 112.8)
- C38: value 10uF -> 100 uF; footprint Capacitor_SMD:C_0603_1608Metric -> Capacitor_SMD:CP_Elec_5x5.3
- moved C38 33.0 mm to (175.3, 143.0)
- moved R32 31.3 mm to (105.2, 122.8), turned to 90 degrees
- moved D10 21.9 mm to (133.6, 116.0), turned to 180 degrees
- moved R48 21.4 mm to (136.1, 115.7)
- moved R17 17.2 mm to (100.4, 111.2), turned to 180 degrees
- moved R16 15.9 mm to (100.4, 110.2), turned to 180 degrees
- moved R39 15.4 mm to (138.1, 113.8)
- moved R49 15.4 mm to (136.1, 113.8)
- moved D13 15.2 mm to (133.6, 125.5), turned to 180 degrees
- moved D15 15.2 mm to (133.6, 114.1)
- moved R45 14.3 mm to (136.1, 125.2), turned to 180 degrees
- moved R36 13.7 mm to (138.1, 108.0)
- moved R41 13.7 mm to (136.1, 108.0)
- moved D11 13.5 mm to (133.6, 108.3)
- moved R10 12.7 mm to (142.7, 106.2)
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Connections:
- C38 pad 1: +5V -> +3V3
- C48 pad 1: /3V3_PCIE -> +3V3
- C51 pad 1: /3V3_PCIE -> +3V3
- J2 pad 10: /RUN_PG -> GND
- J2 pad 11: /KSZ_RESETN -> /nRPIBOOT
- J2 pad 12: /nEXTRST -> GND
- J2 pad 13: Net-(J2-Pad13) -> /GLOBAL_EN
- J2 pad 14: Net-(J2-Pad14) -> GND
- J2 pad 16: Net-(J2-Pad16) -> GND
- J2 pad 3: GND -> /nEXTRST
- J2 pad 4: /nRPIBOOT -> /KSZ_RESETN
- J2 pad 5: GND -> Net-(J2-Pad5)
- J2 pad 6: /GLOBAL_EN -> Net-(J2-Pad6)
- J2 pad 7: GND -> /RUN_PG
- J2 pad 8: /LED_PWR -> GND
- J2 pad 9: GND -> /LED_PWR
- R54 pad 1: /3V3_PCIE -> +3V3
- TP3 pad 1: /3V3_PCIE -> +3V3
- U1 pad 47: Net-(U1-Pad47) -> /INTRP_N
- U10 pad 12: /3V3_PCIE -> +3V3
- U10 pad 14: /3V3_PCIE -> +3V3
- U10 pad 16: /3V3_PCIE -> +3V3
- U10 pad 18: /3V3_PCIE -> +3V3
- U10 pad 2: /3V3_PCIE -> +3V3
- U10 pad 4: /3V3_PCIE -> +3V3
- U10 pad 70: /3V3_PCIE -> +3V3
- U10 pad 72: /3V3_PCIE -> +3V3
- U10 pad 74: /3V3_PCIE -> +3V3
- U2 pad 95: Net-(R22-Pad1) -> /SYN_CLKO
- U5 pad 2: /3V3_PCIE -> +3V3
Routing:
- net GND: track 61.7 -> 344.3 mm, vias 66 -> 272
- net +5V: track 143.2 -> 250.4 mm, vias 12 -> 32
- net /SFP_I2C_SDA: track 12.1 -> 72.3 mm, vias 0 -> 2
- net /SFP_I2C_SCL: track 11.7 -> 71.0 mm
- net /KSZ_RESETN: track 0.00 -> 46.4 mm, vias 0 -> 2
- net /EEPROM_nWP: track 0.00 -> 44.4 mm
- net /INTRP_N: track 0.00 -> 38.5 mm, vias 0 -> 2
- net +3V3: track 29.6 -> 65.6 mm, vias 11 -> 60
- net /RPI_UART_TX: track 0.00 -> 35.3 mm, vias 0 -> 1
- net /MISO: track 0.00 -> 34.9 mm, vias 0 -> 2
- net Net-(R55-Pad2): track 0.00 -> 31.8 mm, vias 0 -> 2
- net /MOSI: track 0.00 -> 31.2 mm, vias 0 -> 2
- net /SCS: track 0.00 -> 31.1 mm, vias 0 -> 2
- net /LED4_0: track 0.00 -> 31.1 mm, vias 0 -> 2
- net /SCLK: track 0.00 -> 30.6 mm, vias 0 -> 2
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- added copper zone on B.Cu, net +3V3
- added copper zone on In2.Cu, net +3V3
- added copper zone on In1.Cu, net GND
- removed copper zone on F.Cu, net (none)
- removed copper zone on F.Cu, net /3V3_PCIE
Other:
- outline, holes or cut-outs redrawn
