File: switch-test-board/switch-test-board.sch (KiCad schematic (older format))
At the start: 201 parts, among them J1 USB_B_Micro, J2 2011-2X10G00SD025B, J3 1367073-1, J4 2011-2X10G00SD025B, SW1 PTS645SM43SMTR92 LFS, U1 RPI4CM, U10 MDT420M02001, U2 KSZ9477S, U3 LD39200PUR, U4 piSlice-PCIe-X1-Conn, U5 LM1085ISX-3.3/NOPB, U6 LD39200PUR, U7 LD39200PUR, U8 piSlice-PCIe-X1-Edge, U9 MIC826TYMT, Y1 ABM8G-25.000MHZ-B4Y-T

Commit message: PCB updated.
Parts:
- removed C45: 10uF, Capacitor_SMD:C_0603_1608Metric, symbol Device:C_Small
- removed FB3: BLM18EG221SN1D, kicad-lib:ferrite-blm18, symbol Device:Ferrite_Bead_Small
- added C100, C101, C102, C99: 0.1uF, Capacitor_SMD:C_0402_1005Metric, symbol Device:C_Small
- added FB8: BLM18EG221SN1D, kicad-lib:ferrite-blm18, symbol Device:Ferrite_Bead_Small
- added J5: JK0654219, Connector_RJ:RJ45_Pulse_JK0654219NL_Horizontal, symbol Connector:JK0654219
Connections:
- net labels added: GNDREF, P4_TXRX_A_N, P4_TXRX_A_P, P4_TXRX_B_N, P4_TXRX_B_P, P4_TXRX_C_N, P4_TXRX_C_P, P4_TXRX_D_N, P4_TXRX_D_P, RPI_USBD_N, RPI_USBD_P
- net labels removed: DVDDL_1V2, RPI_USB_DM, RPI_USB_DP
- wire segments 826 -> 850

Commit message: PCB Design Completed.
Parts:
- removed C49: 0.1uF, Capacitor_SMD:C_0402_1005Metric, symbol Device:C_Small
- removed C50, C54: 10uF, Capacitor_SMD:C_0603_1608Metric, symbol Device:C_Small
- removed J4: 2011-2X10G00SD025B, Connector_PinHeader_2.54mm:PinHeader_2x10_P2.54mm_Vertical, symbol Connector_Generic:Conn_02x10_Odd_Even
- removed R22: 22R, Resistor_SMD:R_0402_1005Metric, symbol Device:R_Small_US
- removed R30: 56K, Resistor_SMD:R_0402_1005Metric, symbol Device:R_Small_US
- removed R31: 10K, Resistor_SMD:R_0402_1005Metric, symbol Device:R_Small_US
- removed TP4: TestPoint, TestPoint:TestPoint_Pad_D1.0mm, symbol Connector:TestPoint
- removed U3: LD39200PUR, Package_DFN_QFN:DFN-6-1EP_3x3mm_P0.95mm_EP1.7x2.6mm, symbol kicad-lib:LD39200PUR
- added R56, R57, R58, R59, R60, R61, R62, R63, R64: 0R_DNP, Resistor_SMD:R_0402_1005Metric, symbol Device:R_Small_US
- C38: value 10uF -> 100 uF; footprint Capacitor_SMD:C_0603_1608Metric -> Capacitor_SMD:CP_Elec_5x5.3; Part Number (none) -> 865080142007
Connections:
- wire segments 850 -> 833
- no-connect marks 47 -> 46
